File: circuit/circuit.kicad_sch (KiCad schematic)
At the start: 1 part, among them U1 Pico

Commit message: .
Parts:
- added D1, D2, D3, D4: LED, symbol Device:LED
- added J1: Sensors, symbol Connector_Generic:Conn_01x05
- added K1: Relay_SPDT, symbol Relay:Relay_SPDT
- added R1, R2, R3, R4: R, symbol Device:R
- added SW1: Motor On, symbol Switch:SW_Push
- added SW2: Motor Off, symbol Switch:SW_Push
Connections:
- net at U1.1 (GPIO0): now also D1.2 (A)
- net at U1.19 (GPIO14): now also SW1.2
- net at U1.2 (GPIO1): now also D2.2 (A)
- net at U1.20 (GPIO15): now also SW2.2
- net GND: now reaches U1.23 (GND)
- net GND: now also J1.5 (Pin_5), R1.1, R2.1, R3.1, R4.1, SW1.1, SW2.1
- net at U1.24 (GPIO18): now also J1.4 (Pin_4)
- net at U1.25 (GPIO19): now also J1.3 (Pin_3)
- net at U1.26 (GPIO20): now also J1.2 (Pin_2)
- net at U1.27 (GPIO21): now also J1.1 (Pin_1)
- net at U1.34 (GPIO28_ADC2): now also K1.A2
- net at U1.4 (GPIO2): now also D3.2 (A)
- net at U1.5 (GPIO3): now also D4.2 (A)
- new net: D4.1 (K), R4.2
- new net: D3.1 (K), R3.2
- new net: D1.1 (K), R1.2
- new net: D2.1 (K), R2.2
